Commit message: fix: adjust gripper positions so it works properly on ignition

File: interbotix_ros_xsarms/interbotix_xsarm_descriptions/urdf/vx300s.urdf.xacro (robot description, xacro)
@@ -593,7 +593,10 @@
         <link name="$(arg robot_name)/left_finger_link">
           <visual>
+            <!-- <origin
+              rpy="${pi/2} ${-pi} ${pi/2}"
+              xyz="-0.0404 -0.0575 0"/> -->
             <origin
               rpy="${pi/2} ${-pi} ${pi/2}"
-              xyz="-0.0404 -0.0575 0"/>
+              xyz="-0.0404 -0.025 0"/>
             <geometry>
               <mesh
@@ -604,7 +607,10 @@
           </visual>
           <collision>
+            <!-- <origin
+              rpy="${pi/2} ${-pi} ${pi/2}"
+              xyz="-0.0404 -0.0575 0"/> -->
             <origin
               rpy="${pi/2} ${-pi} ${pi/2}"
-              xyz="-0.0404 -0.0575 0"/>
+              xyz="-0.0404 -0.025 0"/>
             <geometry>
               <mesh
@@ -653,7 +659,10 @@
         <link name="$(arg robot_name)/right_finger_link">
           <visual>
+            <!-- <origin
+              rpy="${-pi/2} ${pi} ${-pi/2}"
+              xyz="-0.0404 0.0575 0 "/> -->
             <origin
               rpy="${-pi/2} ${pi} ${-pi/2}"
-              xyz="-0.0404 0.0575 0 "/>
+              xyz="-0.0404 0.025 0 "/>
             <geometry>
               <mesh
@@ -664,7 +673,10 @@
           </visual>
           <collision>
+            <!-- <origin
+              rpy="${-pi/2} ${pi} ${-pi/2}"
+              xyz="-0.0404 0.0575 0 "/> -->
             <origin
               rpy="${-pi/2} ${pi} ${-pi/2}"
-              xyz="-0.0404 0.0575 0 "/>
+              xyz="-0.0404 0.025 0 "/>
             <geometry>
               <mesh

Commit message: restore original vx300s urdf

File: interbotix_ros_xsarms/interbotix_xsarm_descriptions/urdf/vx300s.urdf.xacro (robot description, xacro)
@@ -47,5 +47,5 @@
   <xacro:property name="finger_limit_effort"        value="5"/>
   <xacro:property name="finger_limit_lower"         value="0.021"/>
-  <xacro:property name="finger_limit_upper"         value="0.077"/>
+  <xacro:property name="finger_limit_upper"         value="0.057"/>
   <xacro:property name="finger_limit_vel"           value="1"/>
   <material name="interbotix_black">
@@ -577,5 +577,5 @@
           <limit
             effort="${finger_limit_effort}"
-            lower="-${finger_limit_lower}"
+            lower="${finger_limit_lower}"
             upper="${finger_limit_upper}"
             velocity="${finger_limit_vel}"/>
@@ -595,5 +595,5 @@
             <origin
               rpy="${pi/2} ${-pi} ${pi/2}"
-              xyz="-0.0404 -0.025 0"/>
+              xyz="-0.0404 -0.0575 0"/>
             <geometry>
               <mesh
@@ -606,5 +606,5 @@
             <origin
               rpy="${pi/2} ${-pi} ${pi/2}"
-              xyz="-0.0404 -0.025 0"/>
+              xyz="-0.0404 -0.0575 0"/>
             <geometry>
               <mesh
@@ -631,6 +631,6 @@
           <limit
             effort="${finger_limit_effort}"
-            lower="-${finger_limit_upper}"
-            upper="${finger_limit_lower}"
+            lower="${-finger_limit_upper}"
+            upper="${-finger_limit_lower}"
             velocity="${finger_limit_vel}"/>
           <origin
@@ -655,5 +655,5 @@
             <origin
               rpy="${-pi/2} ${pi} ${-pi/2}"
-              xyz="-0.0404 0.025 0 "/>
+              xyz="-0.0404 0.0575 0 "/>
             <geometry>
               <mesh
@@ -666,5 +666,5 @@
             <origin
               rpy="${-pi/2} ${pi} ${-pi/2}"
-              xyz="-0.0404 0.025 0 "/>
+              xyz="-0.0404 0.0575 0 "/>
             <geometry>
               <mesh
