Commit message: fix(interbotix_ros_xsarms): changed to be compatible with moveit

File: interbotix_ros_xsarms/interbotix_xsarm_descriptions/urdf/control.urdf.xacro (robot description, xacro)
@@ -86,6 +86,6 @@
         <xacro:if value="${hardware_type == 'gz_classic'}">
           <joint name="right_finger">
-            <param name="mimic">left_finger</param>
-            <param name="multiplier">1</param>
+            <!-- <param name="mimic">left_finger</param>
+            <param name="multiplier">1</param> -->
             <command_interface name="position">
               <param name="min">"${-finger_limit_lower}"</param>

File: interbotix_ros_xsarms/interbotix_xsarm_descriptions/urdf/vx300s.urdf.xacro (robot description, xacro)
@@ -47,5 +47,5 @@
   <xacro:property name="finger_limit_effort"        value="5"/>
   <xacro:property name="finger_limit_lower"         value="0.021"/>
-  <xacro:property name="finger_limit_upper"         value="0.057"/>
+  <xacro:property name="finger_limit_upper"         value="0.077"/>
   <xacro:property name="finger_limit_vel"           value="1"/>
   <material name="interbotix_black">
@@ -577,5 +577,5 @@
           <limit
             effort="${finger_limit_effort}"
-            lower="${finger_limit_lower}"
+            lower="-${finger_limit_lower}"
             upper="${finger_limit_upper}"
             velocity="${finger_limit_vel}"/>
@@ -595,5 +595,5 @@
             <origin
               rpy="${pi/2} ${-pi} ${pi/2}"
-              xyz="-0.0404 -0.0575 0"/>
+              xyz="-0.0404 -0.025 0"/>
             <geometry>
               <mesh
@@ -606,5 +606,5 @@
             <origin
               rpy="${pi/2} ${-pi} ${pi/2}"
-              xyz="-0.0404 -0.0575 0"/>
+              xyz="-0.0404 -0.025 0"/>
             <geometry>
               <mesh
@@ -631,6 +631,6 @@
           <limit
             effort="${finger_limit_effort}"
-            lower="${-finger_limit_upper}"
-            upper="${-finger_limit_lower}"
+            lower="-${finger_limit_upper}"
+            upper="${finger_limit_lower}"
             velocity="${finger_limit_vel}"/>
           <origin
@@ -655,5 +655,5 @@
             <origin
               rpy="${-pi/2} ${pi} ${-pi/2}"
-              xyz="-0.0404 0.0575 0 "/>
+              xyz="-0.0404 0.025 0 "/>
             <geometry>
               <mesh
@@ -666,5 +666,5 @@
             <origin
               rpy="${-pi/2} ${pi} ${-pi/2}"
-              xyz="-0.0404 0.0575 0 "/>
+              xyz="-0.0404 0.025 0 "/>
             <geometry>
               <mesh

Commit message: tmnc

File: interbotix_ros_xsarms/interbotix_xsarm_descriptions/urdf/control.urdf.xacro (robot description, xacro)
@@ -18,5 +18,6 @@
       <!-- If simulating the robot in Gazebo Classic -->
       <xacro:if value="${hardware_type == 'gz_classic'}">
-        <plugin>gazebo_ros2_control/GazeboSystem</plugin>
+        <!-- <plugin>ign_ros2_control/IgnitionSystem</plugin> -->
+        <plugin>gz_ros2_control/GazeboSimSystem</plugin>
       </xacro:if>
     </hardware>
@@ -99,5 +100,5 @@
   <xacro:if value="${hardware_type == 'gz_classic'}">
     <gazebo>
-      <!-- <plugin filename="libgazebo_ros2_control.so" name="gazebo_ros2_control">
+      <!-- <plugin filename="libign_ros2_control-system.so" name="ign_ros2_control::IgnitionROS2ControlPlugin">
         <ros>
           <namespace>/$(arg robot_name)</namespace>

File: interbotix_ros_xsarms/interbotix_xsarm_descriptions/urdf/vx300s.urdf.xacro (robot description, xacro)
@@ -47,5 +47,5 @@
   <xacro:property name="finger_limit_effort"        value="5"/>
   <xacro:property name="finger_limit_lower"         value="0.021"/>
-  <xacro:property name="finger_limit_upper"         value="0.057"/>
+  <xacro:property name="finger_limit_upper"         value="0.077"/>
   <xacro:property name="finger_limit_vel"           value="1"/>
   <material name="interbotix_black">
@@ -577,5 +577,5 @@
           <limit
             effort="${finger_limit_effort}"
-            lower="${finger_limit_lower}"
+            lower="-${finger_limit_lower}"
             upper="${finger_limit_upper}"
             velocity="${finger_limit_vel}"/>
@@ -595,5 +595,5 @@
             <origin
               rpy="${pi/2} ${-pi} ${pi/2}"
-              xyz="-0.0404 -0.0575 0"/>
+              xyz="-0.0404 -0.025 0"/>
             <geometry>
               <mesh
@@ -606,5 +606,5 @@
             <origin
               rpy="${pi/2} ${-pi} ${pi/2}"
-              xyz="-0.0404 -0.0575 0"/>
+              xyz="-0.0404 -0.025 0"/>
             <geometry>
               <mesh
@@ -627,10 +627,10 @@
           </inertial>
         </link>
-        <joint name="right_finger" type="prismatic">
+        <joint name="right_finger_mimic" type="prismatic">
           <axis xyz="0 1 0"/>
           <limit
             effort="${finger_limit_effort}"
-            lower="${-finger_limit_upper}"
-            upper="${-finger_limit_lower}"
+            lower="-${finger_limit_upper}"
+            upper="${finger_limit_lower}"
             velocity="${finger_limit_vel}"/>
           <origin
@@ -650,4 +650,10 @@
               offset="0"/>
           </xacro:if>
+          <xacro:if value="${hardware_type == 'gz_classic'}">
+            <mimic
+              joint="left_finger"
+              multiplier="-1"
+              offset="0"/>
+          </xacro:if>
         </joint>
         <link name="$(arg robot_name)/right_finger_link">
@@ -655,5 +661,5 @@
             <origin
               rpy="${-pi/2} ${pi} ${-pi/2}"
-              xyz="-0.0404 0.0575 0 "/>
+              xyz="-0.0404 0.025 0 "/>
             <geometry>
               <mesh
@@ -666,5 +672,5 @@
             <origin
               rpy="${-pi/2} ${pi} ${-pi/2}"
-              xyz="-0.0404 0.0575 0 "/>
+              xyz="-0.0404 0.025 0 "/>
             <geometry>
               <mesh

Commit message: fix(right finger): fix right finger mimic in simulation

File: interbotix_ros_xsarms/interbotix_xsarm_descriptions/urdf/control.urdf.xacro (robot description, xacro)
@@ -85,6 +85,7 @@
         <xacro:if value="${hardware_type == 'gz_classic'}">
           <joint name="right_finger">
-            <param name="mimic">left_finger</param>
-            <param name="multiplier">-1</param>
+            <!-- <mimic joint="left_finger" multiplier="-1" offset="0.0"/> -->
+            <!-- <param name="mimic">left_finger</param>
+            <param name="multiplier">-1</param> -->
             <command_interface name="position">
               <param name="min">"${-finger_limit_lower}"</param>
