Commit message: set proper initial states and mimic joint for gripper fingers

File: interbotix_ros_xsarms/interbotix_xsarm_descriptions/urdf/control.urdf.xacro (robot description, xacro)
@@ -17,5 +17,5 @@
       <!-- If simulating the robot in Gazebo Classic -->
       <xacro:if value="${hardware_type == 'gz_classic'}">
-        <plugin>gazebo_ros2_control/GazeboSystem</plugin>
+        <plugin>gz_ros2_control/GazeboSimSystem</plugin>
       </xacro:if>
     </hardware>
@@ -25,5 +25,7 @@
         <param name="max">"${waist_limit_upper}"</param>
       </command_interface>
-      <state_interface name="position"/>
+      <state_interface name="position">
+        <param name="initial_value">0.0</param>
+      </state_interface>
     </joint>
     <joint name="shoulder">
@@ -32,5 +34,7 @@
         <param name="max">"${shoulder_limit_upper}"</param>
       </command_interface>
-      <state_interface name="position"/>
+      <state_interface name="position">
+        <param name="initial_value">-1.50</param>
+      </state_interface>
     </joint>
     <joint name="elbow">
@@ -39,5 +43,7 @@
         <param name="max">"${elbow_limit_upper}"</param>
       </command_interface>
-      <state_interface name="position"/>
+      <state_interface name="position">
+        <param name="initial_value">1.55</param>
+      </state_interface>
     </joint>
     <xacro:if value="${dof >= 6}">
@@ -47,5 +53,7 @@
           <param name="max">"${forearm_roll_limit_upper}"</param>
         </command_interface>
-        <state_interface name="position"/>
+        <state_interface name="position">
+          <param name="initial_value">0.0</param>
+        </state_interface>
       </joint>
     </xacro:if>
@@ -55,5 +63,7 @@
         <param name="max">"${wrist_angle_limit_upper}"</param>
       </command_interface>
-      <state_interface name="position"/>
+      <state_interface name="position">
+        <param name="initial_value">0.5</param>
+      </state_interface>
     </joint>
     <xacro:if value="${dof >= 5}">
@@ -63,5 +73,7 @@
           <param name="max">"${wrist_rotate_limit_upper}"</param>
         </command_interface>
-        <state_interface name="position"/>
+        <state_interface name="position">
+          <param name="initial_value">0.0</param>
+        </state_interface>
       </joint>
     </xacro:if>
@@ -74,36 +86,38 @@
       </xacro:if>
       <xacro:if value="$(arg show_gripper_fingers)">
+        <!-- Main Finger -->
         <joint name="left_finger">
           <command_interface name="position">
             <param name="min">"${finger_limit_lower}"</param>
-            <param name="max">"${-finger_limit_lower}"</param>
+            <param name="max">"${finger_limit_upper}"</param>
           </command_interface>
-          <state_interface name="position"/>
+          <state_interface name="position">
+            <!-- Add this to spawn inside the valid limits -->
+            <param name="initial_value">0.021</param>
+          </state_interface>
+          <!-- <state_interface name="velocity"/> -->
         </joint>
-        <xacro:if value="${hardware_type == 'gz_classic'}">
-          <joint name="right_finger">
-            <!-- <param name="mimic">left_finger</param>
-            <param name="multiplier">1</param> -->
-            <command_interface name="position">
-              <param name="min">"${-finger_limit_lower}"</param>
-              <param name="max">"${finger_limit_lower}"</param>
-            </command_interface>
-            <state_interface name="position"/>
-          </joint>
-        </xacro:if>
+        <!-- Mimic Finger -->
+        <joint name="right_finger">
+          <param name="mimic">left_finger</param>
+          <param name="multiplier">-1.0</param>
+          <!-- We MUST have a command interface for gz_ros2_control to actuate this joint -->
+          <command_interface name="position"/>
+          <state_interface name="position">
+            <!-- Spawn inside the valid [-0.057, -0.021] limits to prevent physics explosions -->
+            <param name="initial_value">-0.021</param>
+          </state_interface>
+        </joint>
       </xacro:if>
     </xacro:if>
   </ros2_control>
-  <!-- Load the gazebo_ros2_control plugin if using Gazebo hardware -->
+  <!-- The robot-level Gazebo plugin is provided by the Clearpath platform xacro
+       (see clearpath_platform_description/urdf/generic/gazebo.urdf.xacro). Do not
+       add a second gz_ros2_control plugin here for gz_classic, because it loads the
+       wrong library and prevents the controller manager from exposing the joints.
+  -->
   <xacro:if value="${hardware_type == 'gz_classic'}">
     <gazebo>
-      <plugin filename="libgazebo_ros2_control.so" name="gazebo_ros2_control">
-        <ros>
-          <namespace>/$(arg robot_name)</namespace>
-        </ros>
-        <robot_param>robot_description</robot_param>
-        <robot_param_node>robot_state_publisher</robot_param_node>
-        <parameters>$(find interbotix_xsarm_sim)/config/trajectory_controllers/${robot_model}_trajectory_controllers.yaml</parameters>
-      </plugin>
+      <!-- intentionally left blank: plugin is provided by the platform-level gz plugin -->
     </gazebo>
     <xacro:include filename="$(find interbotix_common_sim)/media/materials/scripts/interbotix_texture.gazebo"/>

File: interbotix_ros_xsarms/interbotix_xsarm_descriptions/urdf/vx300s.urdf.xacro (robot description, xacro)
@@ -644,10 +644,11 @@
             friction="0.1"
             damping="0.1"/>
-          <xacro:if value="${hardware_type != 'gz_classic'}">
+          <!-- <xacro:if value="${hardware_type != 'gz_classic'}">
             <mimic
               joint="left_finger"
               multiplier="-1"
               offset="0"/>
-          </xacro:if>
+          </xacro:if> -->
+          <mimic joint="left_finger" multiplier="-1" offset="0"/>
         </joint>
         <link name="$(arg robot_name)/right_finger_link">

Commit message: feat(xsarm_descriptions): gazebo initial values, gripper joints out of the gz arm block

File: interbotix_ros_xsarms/interbotix_xsarm_descriptions/urdf/control.urdf.xacro (robot description, xacro)
@@ -18,6 +18,4 @@
       <!-- If simulating the robot in Gazebo Classic -->
       <xacro:if value="${hardware_type == 'gz_classic'}">
-        <!-- <plugin>gazebo_ros2_control/GazeboSystem</plugin> -->
-        <!-- <plugin>ign_ros2_control/IgnitionSystem</plugin> -->
         <plugin>gz_ros2_control/GazeboSimSystem</plugin>
       </xacro:if>
@@ -28,5 +26,7 @@
         <param name="max">"${waist_limit_upper}"</param>
       </command_interface>
-      <state_interface name="position"/>
+      <state_interface name="position">
+        <param name="initial_value">0.0</param>
+      </state_interface>
     </joint>
     <joint name="shoulder">
@@ -35,5 +35,7 @@
         <param name="max">"${shoulder_limit_upper}"</param>
       </command_interface>
-      <state_interface name="position"/>
+      <state_interface name="position">
+        <param name="initial_value">-1.50</param>
+      </state_interface>
     </joint>
     <joint name="elbow">
@@ -42,5 +44,7 @@
         <param name="max">"${elbow_limit_upper}"</param>
       </command_interface>
-      <state_interface name="position"/>
+      <state_interface name="position">
+        <param name="initial_value">1.55</param>
+      </state_interface>
     </joint>
     <xacro:if value="${dof >= 6}">
@@ -50,5 +54,7 @@
           <param name="max">"${forearm_roll_limit_upper}"</param>
         </command_interface>
-        <state_interface name="position"/>
+        <state_interface name="position">
+          <param name="initial_value">0.0</param>
+        </state_interface>
       </joint>
     </xacro:if>
@@ -58,5 +64,7 @@
         <param name="max">"${wrist_angle_limit_upper}"</param>
       </command_interface>
-      <state_interface name="position"/>
+      <state_interface name="position">
+        <param name="initial_value">0.5</param>
+      </state_interface>
     </joint>
     <xacro:if value="${dof >= 5}">
@@ -66,9 +74,18 @@
           <param name="max">"${wrist_rotate_limit_upper}"</param>
         </command_interface>
-        <state_interface name="position"/>
+        <state_interface name="position">
+          <param name="initial_value">0.0</param>
+        </state_interface>
       </joint>
     </xacro:if>
     <xacro:if value="$(arg use_gripper)">
-      <xacro:if value="${hardware_type in ('fake', 'gz_classic')}">
+      <!-- Gazebo (gz_classic): the gripper joints are NOT in this block. They have their own
+           ros2_control block, GripperHardwareInterface, in
+           misskal_description/urdf/control/ros2_control.urdf.xacro (arm / gimbal / gripper split).
+           actual: identical to the robot (feat/gripper_controller).
+           TODO(real): stage E3 removes left_finger and gripper_name from the actual block (the
+           gripper moves to misskal_gripper_node); needs the XSHardwareInterface patch first.
+           See misskal_sim study/gripper_sim_integration/TODO_REAL.md (TR-01, TR-08). -->
+      <xacro:if value="${hardware_type == 'fake'}">
         <joint name="gripper">
           <command_interface name="position"/>
@@ -76,25 +93,16 @@
         </joint>
       </xacro:if>
-      <xacro:if value="$(arg show_gripper_fingers)">
-        <joint name="left_finger">
-          <command_interface name="position">
-            <param name="min">"${finger_limit_lower}"</param>
-            <param name="max">"${-finger_limit_lower}"</param>
-          </command_interface>
-          <state_interface name="position"/>
-          <state_interface name="effort"/>
-          <state_interface name="velocity">
-            <param name="initial_value">0.0</param>
-          </state_interface>
-        </joint>
-        <xacro:if value="${hardware_type == 'gz_classic'}">
-          <joint name="right_finger">
-            <!-- <param name="mimic">left_finger</param>
-            <param name="multiplier">1</param> -->
+      <xacro:if value="${hardware_type != 'gz_classic'}">
+        <xacro:if value="$(arg show_gripper_fingers)">
+          <joint name="left_finger">
             <command_interface name="position">
-              <param name="min">"${-finger_limit_lower}"</param>
-              <param name="max">"${finger_limit_lower}"</param>
+              <param name="min">"${finger_limit_lower}"</param>
+              <param name="max">"${-finger_limit_lower}"</param>
             </command_interface>
             <state_interface name="position"/>
+            <state_interface name="effort"/>
+            <state_interface name="velocity">
+              <param name="initial_value">0.0</param>
+            </state_interface>
           </joint>
         </xacro:if>
@@ -102,15 +110,12 @@
     </xacro:if>
   </ros2_control>
-  <!-- Load the gazebo_ros2_control plugin if using Gazebo hardware -->
+  <!-- The robot-level Gazebo plugin is provided by the Clearpath platform xacro
+       (see clearpath_platform_description/urdf/generic/gazebo.urdf.xacro). Do not
+       add a second gz_ros2_control plugin here for gz_classic, because it loads the
+       wrong library and prevents the controller manager from exposing the joints.
+  -->
   <xacro:if value="${hardware_type == 'gz_classic'}">
     <gazebo>
-      <!-- <plugin filename="libgazebo_ros2_control.so" name="gazebo_ros2_control">
-        <ros>
-          <namespace>/$(arg robot_name)</namespace>
-        </ros>
-        <robot_param>robot_description</robot_param>
-        <robot_param_node>robot_state_publisher</robot_param_node>
-        <parameters>$(find interbotix_xsarm_sim)/config/trajectory_controllers/${robot_model}_trajectory_controllers.yaml</parameters>
-      </plugin> -->
+      <!-- intentionally left blank: plugin is provided by the platform-level gz plugin -->
     </gazebo>
     <xacro:include filename="$(find interbotix_common_sim)/media/materials/scripts/interbotix_texture.gazebo"/>

File: interbotix_ros_xsarms/interbotix_xsarm_descriptions/urdf/vx300s.urdf.xacro (robot description, xacro)
@@ -644,10 +644,11 @@
             friction="0.1"
             damping="0.1"/>
-          <xacro:if value="${hardware_type != 'gz_classic'}">
+          <!-- <xacro:if value="${hardware_type != 'gz_classic'}">
             <mimic
               joint="left_finger"
               multiplier="-1"
               offset="0"/>
-          </xacro:if>
+          </xacro:if> -->
+          <mimic joint="left_finger" multiplier="-1" offset="0"/>
         </joint>
         <link name="$(arg robot_name)/right_finger_link">
